Commit message: Fixed the problem with the definition of the kfe joint limits

File: gazebo/gazebo.urdf.xacro (robot description, xacro)
@@ -4,5 +4,5 @@
 		<plugin name="gazebo_ros_controller_manager" filename="libgazebo_ros_control.so">
 			<robotNamespace>/hyq2max</robotNamespace>
-			<controlPeriod>0.001</controlPeriod>
+			<controlPeriod>0.005</controlPeriod>
 		</plugin>
 		<plugin filename="libgazebo_ros_p3d.so" name="gazebo_ros_p3d">

File: robots/hyq2max.urdf.xacro (robot description, xacro)
@@ -17,5 +17,5 @@
 	<!-- Generic simulator_gazebo plugins for starting mechanism control, ros time -->
 	<xacro:include filename="$(find hyq2max_description)/gazebo/gazebo.urdf.xacro"/>
-	<!-- Now we can start using the macros included above to define the actual HyQ -->
+	<!-- Now we can start using the macros included above to define the actual HyQ2Max -->
 	<!-- The first use of a macro. This one was defined in trunk.urdf.xacro above.
 A macro like this will expand to a set of link and joint definitions, and to additional
@@ -25,6 +25,6 @@
 the origin block defines where the component is w.r.t its parent (in this case the parent
 is the world frame). For more, see http://www.ros.org/wiki/xacro -->
-	<!-- body -->
-	<!-- torso -->
+	<!-- Body -->
+	<!-- Trunk -->
 	<xacro:hyq2max_trunk name="base">
 		<origin xyz="-0.443 -0.191 -0.276" rpy="0 0 0"/>
@@ -34,36 +34,34 @@
 		name="lf"
 		parent="trunk"
-		reflect_hip="1"
-		reflect_upper="1"
+		reflect_left="1"
 		reflect_front="1">
-		<origin xyz="${d_fh/2} ${d_lr/2} 0" rpy="0 ${PI/2} ${PI}"/>
+		<origin xyz="0.4435 0.097 0" rpy="${PI} ${PI/2} 0"/>
+<!--		<origin xyz="${d_fh/2} ${d_lr/2} 0" rpy="0 ${PI/2} ${PI}"/>-->
 	</xacro:hyq2max_leg>
 	<!-- RF leg -->
-<!--	<xacro:hyq2max_leg
+	<xacro:hyq2max_leg
 		name="rf"
 		parent="trunk"
-		reflect_hip="-1"
-		reflect_upper="-1"
+		reflect_left="-1"
 		reflect_front="1">
-		<origin xyz="${d_fh/2} ${-d_lr/2} 0" rpy="0 ${PI/2} 0"/>
-	</xacro:hyq2max_leg>-->
+		<origin xyz="0.4435 -0.097 0" rpy="0 ${PI/2} 0"/>
+<!--		<origin xyz="${d_fh/2} ${-d_lr/2} 0" rpy="0 ${PI/2} 0"/>-->
+	</xacro:hyq2max_leg>
 	<!-- LH leg -->
-<!--	<xacro:hyq2max_leg
+	<xacro:hyq2max_leg
 		name="lh"
 		parent="trunk"
-		reflect_hip="-1"
-		reflect_upper="1"
+		reflect_left="1"
 		reflect_front="-1">
-		<origin xyz="${-d_fh/2} ${d_lr/2} 0" rpy="0 ${PI/2} ${PI}"/>
-	</xacro:hyq2max_leg>-->
+		<origin xyz="-0.4435 0.097 0" rpy="${PI} ${PI/2} 0"/>
+	</xacro:hyq2max_leg>
 	<!-- RH leg -->
-<!--	<xacro:hyq2max_leg
+	<xacro:hyq2max_leg
 		name="rh"
 		parent="trunk"
-		reflect_hip="1"
-		reflect_upper="-1"
+		reflect_left="-1"
 		reflect_front="-1">
-		<origin xyz="${-d_fh/2} ${-d_lr/2} 0" rpy="0 ${PI/2} 0"/>
-	</xacro:hyq2max_leg>-->
+		<origin xyz="-0.4435 -0.097 0" rpy="0 ${PI/2} 0"/>
+	</xacro:hyq2max_leg>
 	<!-- IMU trunk -->
 <!--	<xacro:microstrain_3dmgx325_imu

File: urdfs/common.xacro (robot description, xacro)
@@ -5,43 +5,51 @@
 	<property name="d_lr" value="0.414"/>
 	<property name="d_fh" value="0.747"/>
-	<property name="d_tbb" value="0.082"/>
-	<property name="d_p1p2" value="0.35"/>
-	<!-- Initial joint positions -->
-	<property name="haa_pos0" value="0"/>
-	<property name="hfe_pos0" value="0"/>
-	<property name="kfe_pos0" value="0"/>
+	<property name="upperleg_length" value="0.1075"/>
+	<property name="lowerleg_length" value="0.364"/>
 	<!-- Inertial values -->
 	<!-- Trunk with hydraulic system -->
-	<property name="m_trunk" value="53.0"/>
-	<property name="ixx_trunk" value="1.26"/>
-	<property name="iyy_trunk" value="6.56"/>
-	<property name="izz_trunk" value="6.69"/>
-	<property name="ixy_trunk" value="0.03"/>
-	<property name="ixz_trunk" value="-0.06"/>
-	<property name="iyz_trunk" value="-0.03"/>
+	<property name="xcom_trunk" value="0.057737"/>
+	<property name="ycom_trunk" value="0.000687"/>
+	<property name="zcom_trunk" value="-0.005584"/>
+	<property name="m_trunk" value="37.31"/>
+	<property name="ixx_trunk" value="0.296767"/>
+	<property name="iyy_trunk" value="4.418458"/>
+	<property name="izz_trunk" value="4.472778"/>
+	<property name="ixy_trunk" value="0.008818"/>
+	<property name="ixz_trunk" value="0.002473"/>
+	<property name="iyz_trunk" value="0.000597"/>
 	<!-- Hip assembly -->
-	<property name="m_hipassembly" value="2.482"/>
-	<property name="ixx_hipassembly" value="0.0956126"/>
-	<property name="iyy_hipassembly" value="0.1012626"/>
-	<property name="izz_hipassembly" value="6.758E-4"/>
-	<property name="ixy_hipassembly" value="0.0"/>
-	<property name="ixz_hipassembly" value="0.011"/>
-	<property name="iyz_hipassembly" value="0.0"/>
+	<property name="xcom_hipassembly" value="-0.000605"/>
+	<property name="ycom_hipassembly" value="-0.001346"/>
+	<property name="zcom_hipassembly" value="0.000196"/>
+	<property name="m_hipassembly" value="3.54"/>
+	<property name="ixx_hipassembly" value="0.007379"/>
+	<property name="iyy_hipassembly" value="0.004284"/>
+	<property name="izz_hipassembly" value="0.007090"/>
+	<property name="ixy_hipassembly" value="0.000053"/>
+	<property name="ixz_hipassembly" value="-0.000017"/>
+	<property name="iyz_hipassembly" value="-0.000030"/>
 	<!-- Upper leg -->
-	<property name="m_upperleg" value="2.16"/>
-	<property name="ixx_upperleg" value="0.004785"/>
-	<property name="iyy_upperleg" value="0.076166"/>
-	<property name="izz_upperleg" value="0.078576"/>
-	<property name="ixy_upperleg" value="0.0071588"/>
-	<property name="ixz_upperleg" value="0.0"/>
-	<property name="iyz_upperleg" value="0.0"/>
+	<property name="xcom_upperleg" value="0.144296"/>
+	<property name="ycom_upperleg" value="-0.002071"/>
+	<property name="zcom_upperleg" value="-0.005094"/>
+	<property name="m_upperleg" value="4.95"/>
+	<property name="ixx_upperleg" value="0.010196"/>
+	<property name="iyy_upperleg" value="0.204183"/>
+	<property name="izz_upperleg" value="0.207532"/>
+	<property name="ixy_upperleg" value="-0.002320"/>
+	<property name="ixz_upperleg" value="-0.000141"/>
+	<property name="iyz_upperleg" value="0.000034"/>
 	<!-- Lower leg -->
-	<property name="m_lowerleg" value="1.8717"/>
-	<property name="ixx_lowerleg" value="9.0E-4"/>
-	<property name="iyy_lowerleg" value="0.0777"/>
-	<property name="izz_lowerleg" value="0.0775"/>
-	<property name="ixy_lowerleg" value="-0.0"/>
-	<property name="ixz_lowerleg" value="-0.0"/>
-	<property name="iyz_lowerleg" value="0.0"/>
+	<property name="xcom_lowerleg" value="0.109015"/>
+	<property name="ycom_lowerleg" value="0.042147"/>
+	<property name="zcom_lowerleg" value="0.000219"/>
+	<property name="m_lowerleg" value="1.71"/>
+	<property name="ixx_lowerleg" value="0.006848"/>
+	<property name="iyy_lowerleg" value="0.055957"/>
+	<property name="izz_lowerleg" value="0.059397"/>
+	<property name="ixy_lowerleg" value="0.011981"/>
+	<property name="ixz_lowerleg" value="0.000008"/>
+	<property name="iyz_lowerleg" value="0.000012"/>
 	<!-- PTU unit -->
 	<property name="pan_velocity" value="1.0" />

File: urdfs/leg/leg.transmission.xacro (robot description, xacro)
@@ -14,5 +14,5 @@
 		</transmission>
     	<!-- Upper leg -->
-		<transmission name="${name}_hfe_upper_trans">
+		<transmission name="${name}_hfe_trans">
 			<type>transmission_interface/SimpleTransmission</type>
 			<joint name="${name}_hfe_joint">

File: urdfs/leg/leg.urdf.xacro (robot description, xacro)
@@ -5,78 +5,68 @@
 	<xacro:include filename="$(find hyq2max_description)/urdfs/leg/leg.gazebo.xacro"/>
 	<!-- ================================== Leg ================================== -->
-	<!-- The xacro macro xacro:hyq_leg contains: hip assembly, upper and lower leg -->
-	<xacro:macro name="hyq2max_leg" params="name parent *origin reflect_hip reflect_upper reflect_front">
+	<!-- The xacro macro xacro:hyq2max_leg contains: hip assembly, upper and lower leg -->
+	<xacro:macro name="hyq2max_leg" params="name parent *origin reflect_left reflect_front">
 		<!-- Joints -->
 		<!-- Hip assembly joint -->
-		<joint name="${name}_haa_assembly_joint" type="fixed">
+		<joint name="${name}_haa_joint" type="revolute">
 			<insert_block name="origin"/>
 			<parent link="${parent}"/>
-			<child  link="${name}_assembly"/>
-		</joint>
-		<!-- Hip joint assembly -->
-		<joint name="${name}_haa_joint" type="revolute">
-			<origin xyz="0 0 0" rpy="0 0 ${haa_pos0}"/>
-			<parent link="${name}_assembly"/>
-			<!--<insert_block name="origin"/>-->
-			<!--<parent link="${parent}"/>-->
-			<child  link="${name}_hip_assembly"/>
-			<limit effort="150.0" velocity="12.0" lower="${-PI/2-haa_pos0}" upper="${PI/6-haa_pos0}"/>
+			<child  link="${name}_hipassembly"/>
 			<axis xyz="0 0 1"/>
 			<dynamics damping="0.1" friction="0" />
-			<safety_controller k_position="100" k_velocity="100" soft_lower_limit="-10" soft_upper_limit="12.45" />
+			<limit effort="150.0" velocity="12.0" lower="${-2*PI/9}" upper="${2*PI/9}"/>
+			<safety_controller k_position="100" k_velocity="100"
+							   soft_lower_limit="-10" soft_upper_limit="12.45" />
 		</joint>
 		<!-- Upper leg joint -->
 		<joint name="${name}_hfe_joint" type="revolute">
-			<origin xyz="${d_tbb} 0.0 0.0" rpy="${reflect_upper*PI/2} ${-reflect_hip*hfe_pos0} 0.0"/>
-			<parent link="${name}_hip_assembly"/>
-			<child  link="${name}_upper_leg"/>
-			<limit effort="150.0" velocity="12.0" lower="${-(1+reflect_front)*5*PI/36-(1-reflect_front)*7*PI/36-reflect_front*hfe_pos0}" upper="${(1-reflect_front)*5*PI/36+(1+reflect_front)*7*PI/36-reflect_front*hfe_pos0}"/>
+			<origin xyz="0 ${-upperleg_length} 0"
+					rpy="${reflect_left*PI/2} 0 0"/>
+			<parent link="${name}_hipassembly"/>
+			<child  link="${name}_upperleg"/>
 			<axis xyz="0 0 1"/>
 			<dynamics damping="0.1" friction="0" />
-			<safety_controller k_position="100" k_velocity="100" soft_lower_limit="-10" soft_upper_limit="12.45" />
+			<limit effort="150.0" velocity="12.0" lower="${-3*PI/4}" upper="${3*PI/4}"/>
+			<safety_controller k_position="100" k_velocity="100"
+							   soft_lower_limit="-10" soft_upper_limit="12.45" />
 		</joint>
 		<!-- Lower leg joint -->
 		<joint name="${name}_kfe_joint" type="revolute">
-			<origin xyz="${d_p1p2} 0 0" rpy="0 0 ${reflect_front*kfe_pos0}"/>
-			<parent link="${name}_upper_leg"/>
-			<child  link="${name}_lower_leg"/>
-			<limit effort="150.0" velocity="12.0" lower="${-(1+reflect_front)*7*PI/18+(1-reflect_front)*PI/18-reflect_front*kfe_pos0}" upper="${(1-reflect_front)*7*PI/18-(1+reflect_front)*PI/18-reflect_front*kfe_pos0}"/>
+			<origin xyz="${lowerleg_length} 0 0" rpy="0 0 0"/>
+			<parent link="${name}_upperleg"/>
+			<child  link="${name}_lowerleg"/>
 			<axis xyz="0 0 1"/>
 			<dynamics damping="0.1" friction="0" />
-			<safety_controller k_position="100" k_velocity="100" soft_lower_limit="-10" soft_upper_limit="12.45" />
+			<limit effort="150.0" velocity="12.0"
+				   lower="${(1-reflect_front)*3*PI/360-(1+reflect_front)*163*PI/360}"
+				   upper="${(1-reflect_front)*163*PI/360-(1+reflect_front)*3*PI/360}"/>
+			<safety_controller k_position="100" k_velocity="100"
+							   soft_lower_limit="-10" soft_upper_limit="12.45" />
+		</joint>
 		<!-- Foot joint -->
-		</joint>
 		<joint name="${name}_foot_joint" type="fixed">
-			<origin xyz="0.34 0 0" rpy="${PI/2} 0 ${-PI/2}"/>
-			<parent link="${name}_lower_leg"/>
+			<origin xyz="0.37432 ${reflect_front*0.066} 0" rpy="${PI/2} 0 ${-PI/2}"/>
+			<parent link="${name}_lowerleg"/>
 			<child  link="${name}_foot"/>
 		</joint>
 		<!-- Links -->
 		<!-- Hip assembly link -->
-		<link name="${name}_assembly">
-			<inertial>
-				<origin xyz="0 0 0"/>
-				<mass value="0.01"/>
-				<inertia ixx="0.01" iyy="0.01" izz="0.01" ixy="0.0" ixz="0.0" iyz="0.0"/>
-			</inertial>
-		</link>
-		<!-- Hip assembly link -->
 		<link name="${name}_hipassembly">
 			<inertial>
-				<origin xyz="0.01310 ${reflect_hip*0.00010} ${reflect_hip*0.05730}"/>
+				<origin xyz="${xcom_hipassembly} ${ycom_hipassembly} ${zcom_hipassembly}"/>
 				<mass value="${m_hipassembly}"/>
 				<inertia ixx="${ixx_hipassembly}" iyy="${iyy_hipassembly}" izz="${izz_hipassembly}"
-						 ixy="${ixy_hipassembly}" ixz="${-reflect_hip*ixz_hipassembly}" iyz="${iyz_hipassembly}"/>
+						 ixy="${ixy_hipassembly}" ixz="${ixz_hipassembly}" iyz="${iyz_hipassembly}"/>
 			</inertial>
 			<visual>
-				<origin xyz="0 0 0" rpy="${(1-reflect_hip)*PI/2} 0 0"/>
+				<origin xyz="0 -0.046 0" rpy="0 ${-PI/2} ${-PI/2}"/><!-- TODO: -0.044 ask Jake -->
 				<geometry>
-					<mesh filename="package://hyq2max_description/meshes/leg/hipassembly.stl" scale="1 1 1"/>
+					<mesh filename="package://hyq2max_description/meshes/leg/hipassembly.dae" scale="1 1 1"/>
 				</geometry>
 			</visual>
 			<collision>
-				<origin xyz="0 0 0" rpy="${(1-reflect_hip)*PI/2} 0 0"/>
+				<origin xyz="0 -0.046 0" rpy="0 ${-PI/2} ${-PI/2}"/><!-- TODO: -0.044 ask Jake -->
 				<geometry>
-					<mesh filename="package://hyq2max_description/meshes/leg/hipassembly.stl" scale="1 1 1"/>
+					<mesh filename="package://hyq2max_description/meshes/leg/hipassembly.dae" scale="1 1 1"/>
 				</geometry>
 			</collision>
@@ -85,19 +75,19 @@
 		<link name="${name}_upperleg">
 			<inertial>
-				<origin xyz="0.14796 ${reflect_upper*0.02958} 0"/>
+				<origin xyz="${xcom_upperleg} ${reflect_front*ycom_upperleg} ${reflect_left*zcom_upperleg}"/>
 				<mass value="${m_upperleg}"/>
 				<inertia ixx="${ixx_upperleg}" iyy="${iyy_upperleg}" izz="${izz_upperleg}"
-						 ixy="${ixy_upperleg}" ixz="${ixz_upperleg}" iyz="${iyz_upperleg}"/>
+						 ixy="${reflect_front*ixy_upperleg}" ixz="${reflect_left*ixz_upperleg}" iyz="${reflect_left*reflect_front*iyz_upperleg}"/>
 			</inertial>
 			<visual>
-				<origin xyz="0 0 0" rpy="${(1-reflect_front)*PI/2} 0 0"/>
+				<origin xyz="0 0 ${-0.03*reflect_left}" rpy="${(1-reflect_left)*PI/2} 0 0"/> <!-- TODO Ask displacement Jake -->
 				<geometry>
-					<mesh filename="package://hyq2max_description/meshes/leg/upperleg.stl" scale="1 1 1"/>
+					<mesh filename="package://hyq2max_description/meshes/leg/upperleg.dae" scale="1 1 1"/>
 				</geometry>
 			</visual>
 			<collision>
-				<origin xyz="0 0 0" rpy="${(1-reflect_front)*PI/2} 0 0"/>
+				<origin xyz="0 0 ${-0.03*reflect_left}" rpy="${(1-reflect_left)*PI/2} 0 0"/> <!-- TODO Ask displacement Jake -->
 				<geometry>
-					<mesh filename="package://hyq2max_description/meshes/leg/upperleg.stl" scale="1 1 1"/>
+					<mesh filename="package://hyq2max_description/meshes/leg/upperleg.dae" scale="1 1 1"/>
 				</geometry>
 			</collision>
@@ -106,18 +96,20 @@
 		<link name="${name}_lowerleg">
 			<inertial>
-				<origin xyz=" 0.17830  0.00030 -0.00010"/>
+				<origin xyz="${xcom_lowerleg} ${reflect_front*ycom_lowerleg} ${reflect_front*zcom_lowerleg}"/>
 				<mass value="${m_lowerleg}"/>
 				<inertia ixx="${ixx_lowerleg}" iyy="${iyy_lowerleg}" izz="${izz_lowerleg}"
-						 ixy="${ixy_lowerleg}" ixz="${ixz_lowerleg}" iyz="${iyz_lowerleg}"/>
+						 ixy="${reflect_front*ixy_lowerleg}" ixz="${reflect_front*ixz_lowerleg}" iyz="${iyz_lowerleg}"/>
 			</inertial>
 			<visual>
+				<origin xyz="0 0 0" rpy="${(1-reflect_front)*PI/2} 0 ${PI}"/> <!-- TODO Ask displacement Jake -->
 				<geometry>
-					<mesh filename="package://hyq2max_description/meshes/leg/lowerleg.stl" scale="1 1 1"/>
+					<mesh filename="package://hyq2max_description/meshes/leg/lowerleg.dae" scale="1 1 1"/>
 				</geometry>
 				<material name="white"/>
 			</visual>
 			<collision>
+				<origin xyz="0 0 0" rpy="${(1-reflect_front)*PI/2} 0 ${PI}"/> <!-- TODO Ask displacement Jake -->
 				<geometry>
-					<mesh filename="package://hyq2max_description/meshes/leg/lowerleg.stl" scale="1 1 1"/>
+					<mesh filename="package://hyq2max_description/meshes/leg/lowerleg.dae" scale="1 1 1"/>
 				</geometry>
 			</collision>

File: urdfs/trunk/trunk.urdf.xacro (robot description, xacro)
@@ -4,6 +4,6 @@
 	<xacro:include filename="$(find hyq2max_description)/urdfs/trunk/trunk.gazebo.xacro"/>
 	<!-- ================================ Trunk ================================ -->
-	<!-- The xacro macro xacro:hyq_base contains: base and torso -->
-	<xacro:macro name="hyq2max_torso" params="name">
+	<!-- The xacro macro xacro:hyq_base contains: base and trunk -->
+	<xacro:macro name="hyq2max_trunk" params="name">
 		<!-- Floating-base Joint -->
 		<joint name="floating_base" type="fixed">
@@ -24,23 +24,24 @@
 		<link name="trunk">
 			<inertial>
-				<origin xyz="-0.00020  0.00010  0.00110"/>
+				<origin xyz="${xcom_trunk} ${ycom_trunk} ${zcom_trunk}"/>
 				<mass value="${m_trunk}"/>
 				<inertia ixx="${ixx_trunk}" iyy="${iyy_trunk}" izz="${izz_trunk}"
 						 ixy="${ixy_trunk}" ixz="${ixz_trunk}" iyz="${iyz_trunk}"/>
 			</inertial>
+			<visual>
+				<origin xyz="0 0 0" rpy="${PI/2} 0 ${PI/2}" />
+				<geometry>
+					<mesh filename="package://hyq2max_description/meshes/trunk/trunk.dae" scale="1 1 1"/>
+				</geometry>
+			</visual>
 			<collision>
+				<origin xyz="0 0 0" rpy="${PI/2} 0 ${PI/2}" />
 				<geometry>
-					<mesh filename="package://hyq2max_description/meshes/trunk/trunk.stl" scale="1 1 1"/>
+					<mesh filename="package://hyq2max_description/meshes/trunk/trunk.dae" scale="1 1 1"/>
 				</geometry>
 			</collision>
-			<visual>
-				<origin xyz="0 0 0" rpy="0 0 0" />
-				<geometry>
-					<mesh filename="package://hyq_description/meshes/trunk/trunk.stl" scale="1 1 1"/>
-				</geometry>
-			</visual>
 		</link>
 		<!-- Extensions -->
-		<xacro:torso_gazebo name="trunk"/>
+		<xacro:trunk_gazebo name="trunk"/>
 	</xacro:macro>
 </robot>
