Commit message: Propagated the changes in the sensor related description from hyq_description repo

File: urdfs/sensors/asus_xtion.urdf.xacro (robot description, xacro)
@@ -9,32 +9,33 @@
 			<insert_block name="origin"/>
 			<parent link="${parent}"/>
-			<child link="${name}_asus_xtion_mount_link"/>
+			<child link="${name}_mount_link"/>
 		</joint>
 		<!-- asus ir sensor physical attachment -->
-		<joint name="${name}_asus_xtion_depth_joint" type="fixed">
+		<joint name="${name}_depth_joint" type="fixed">
 			<origin xyz="${asus_xtion_x} ${asus_xtion_depth_y} ${asus_xtion_z}" rpy="0 0 0"/>
-			<parent link="${name}_asus_xtion_mount_link"/>
-			<child link="${name}_asus_xtion_depth_frame"/>
+			<parent link="${name}_mount_link"/>
+			<child link="${name}_depth_frame"/>
 		</joint>
 		<!-- asus xtion ir sensor frame -->
-		<joint name="${name}_asus_xtion_depth_optical_frame_joint" type="fixed">
-			<origin xyz="0 0 0"	rpy="${asus_xtion_roll} ${asus_xtion_pitch} ${asus_xtion_yaw}"/>
-			<parent link="${name}_asus_xtion_depth_frame"/>
-			<child link="${name}_asus_xtion_depth_optical_frame"/>
+		<joint name="${name}_depth_optical_frame_joint" type="fixed">
+			<origin xyz="${asus_xtion_x} ${asus_xtion_depth_y} ${asus_xtion_z}"
+					rpy="${asus_xtion_roll} ${asus_xtion_pitch} ${asus_xtion_yaw}"/>
+			<parent link="${name}_mount_link"/>
+			<child link="${name}_depth_optical_frame"/>
 		</joint>
 		<!-- asus_xtion rgb sensor physical attachment -->
-		<joint name="${name}_asus_xtion_rgb_joint" type="fixed">
+		<joint name="${name}_rgb_joint" type="fixed">
 			<origin xyz="${asus_xtion_x} ${asus_xtion_rgb_y} ${asus_xtion_z}" rpy="0 0 0"/>
-			<parent link="${name}_asus_xtion_mount_link"/>
-			<child link="${name}_asus_xtion_rgb_frame"/>
+			<parent link="${name}_mount_link"/>
+			<child link="${name}_rgb_frame"/>
 		</joint>
 		<!-- asus xtion rgb sensor frame -->
-		<joint name="${name}_asus_xtion_rgb_optical_frame_joint" type="fixed">
-			<origin xyz="0 0 0"	rpy="${asus_xtion_roll} ${asus_xtion_pitch} ${asus_xtion_yaw}"/>
-			<parent link="${name}_asus_xtion_rgb_frame"/>
-			<child link="${name}_asus_xtion_rgb_optical_frame"/>
+		<joint name="${name}_rgb_optical_frame_joint" type="fixed">
+			<origin xyz="${asus_xtion_x} ${asus_xtion_rgb_y} ${asus_xtion_z}"	rpy="${asus_xtion_roll} ${asus_xtion_pitch} ${asus_xtion_yaw}"/>
+			<parent link="${name}_mount_link"/>
+			<child link="${name}_rgb_optical_frame"/>
 		</joint>
 		<!-- Links -->
-		<link name="${name}_asus_xtion_mount_link">
+		<link name="${name}_mount_link">
 			<inertial>
 				<mass value="0.1"/>
@@ -59,5 +60,5 @@
 		</link>
 		<!-- ir sensor link -->
-		<link name="${name}_asus_xtion_depth_frame">
+		<link name="${name}_depth_frame">
 			<inertial>
 				<mass value="0.1" />
@@ -79,7 +80,7 @@
 		</link>
 		<!-- ir optical sensor link -->
-		<link name="${name}_asus_xtion_depth_optical_frame"/>
+		<link name="${name}_depth_optical_frame"/>
 		<!-- rgb sensor link -->
-		<link name="${name}_asus_xtion_rgb_frame" >
+		<link name="${name}_rgb_frame" >
 			<inertial>
 				<mass value="0.1" />
@@ -101,8 +102,8 @@
 		</link>
 		<!-- rgb optical sensor link -->
-		<link name="${name}_asus_xtion_rgb_optical_frame"/>
+		<link name="${name}_rgb_optical_frame"/>
 	<!-- gazebo extensions -->
-	<xacro:asus_xtion_depth_sensor link_name="${name}_asus_xtion_depth_frame" frame_name="${name}_asus_xtion_depth_optical_frame" camera_name="${name}_asus_xtion" />
-	<xacro:asus_xtion_rgb_sensor link_name="${name}_asus_xtion_rgb_frame" frame_name="${name}_asus_xtion_rgb_optical_frame" camera_name="${name}_asus_xtion" />
+	<xacro:asus_xtion_depth_sensor link_name="${name}_depth_frame" frame_name="${name}_depth_optical_frame" camera_name="${name}"/>
+	<xacro:asus_xtion_rgb_sensor link_name="${name}_rgb_frame" frame_name="${name}_rgb_optical_frame" camera_name="${name}"/>
 	</xacro:macro>
 </root>

File: urdfs/sensors/microstrain_3dmgx325_imu.urdf.xacro (robot description, xacro)
@@ -4,5 +4,6 @@
 	<!-- ============================ IMU microstrain ============================== -->
 	<!-- The xacro macro xacro:microstrain_3dmgx325_imu: imu frame -->
-	<xacro:macro name="microstrain_3dmgx325_imu" params="parent *origin imu_name imu_topic update_rate stdev">
+	<xacro:macro name="microstrain_3dmgx325_imu" params="parent *origin imu_name imu_topic update_rate
+		rate_mean rate_stddev rate_bias_mean rate_bias_stddev accel_mean accel_stddev accel_bias_mean accel_bias_stddev">
 		<!-- Joint -->
 		<joint name="${imu_name}_joint" type="fixed">
@@ -26,5 +27,9 @@
 		</link>
 		<!-- IMU definition -->
-		<xacro:microstrain_3dmgx325_imu_sensor imu_name="${imu_name}" imu_topic="${imu_topic}" update_rate="${update_rate}" stdev="${stdev}"/>
+		<xacro:microstrain_3dmgx325_imu_sensor imu_name="${imu_name}" imu_topic="${imu_topic}"
+		 	update_rate="${update_rate}" rate_mean="${rate_mean}" rate_stddev="${rate_stddev}"
+		 	rate_bias_mean="${rate_bias_mean}" rate_bias_stddev="${rate_bias_stddev}"
+		 	accel_mean="${accel_mean}" accel_stddev="${accel_stddev}" accel_bias_mean="${accel_bias_mean}"
+		 	accel_bias_stddev="${accel_bias_stddev}"/>
 	</xacro:macro>
 </robot>

File: urdfs/sensors/velodyne.urdf.xacro (robot description, xacro)
@@ -6,17 +6,17 @@
 	<xacro:macro name="velodyne" params="name parent *origin">
 		<!-- Joints -->
-		<joint name="${name}_velodyne_joint" type="fixed">
+		<joint name="${name}_joint" type="fixed">
 			<insert_block name="origin"/>
 			<parent link="${parent}"/>
-			<child link="${name}_velodyne_frame"/>
+			<child link="${name}_mount_link"/>
 		</joint>
 		<!-- velodyne sensor optical frame -->
-		<joint name="${name}_velodyne_optical_frame_joint" type="fixed">
+		<joint name="${name}_optical_frame_joint" type="fixed">
 			<origin xyz="${velodyne_x} ${velodyne_y} ${velodyne_z}" rpy="0.0 0.0 0.0"/>
-			<parent link="${name}_velodyne_frame"/>
-			<child link="${name}_velodyne_optical_frame"/>
+			<parent link="${name}_mount_link"/>
+			<child link="${name}"/>
 		</joint>
 		<!-- Links -->
-		<link name="${name}_velodyne_frame">
+		<link name="${name}_mount_link">
 			<inertial>
 				<mass value="0.1"/>
@@ -41,5 +41,5 @@
 		</link>
 		<!-- rgb optical sensor link -->
-		<link name="${name}_velodyne_optical_frame">
+		<link name="${name}">
 			<inertial>
 				<mass value="0.1"/>
@@ -49,5 +49,5 @@
 		</link>
 		<!-- gazebo extensions -->
-		<xacro:velodyne_sensor link_name="${name}_velodyne_optical_frame" frame_name="${name}_velodyne_frame" lidar_name="${name}_velodyne" />
+		<xacro:velodyne_sensor link_name="${name}_optical_frame" frame_name="${name}_frame" lidar_name="${name}" />
 	</xacro:macro>
 </robot>
