Commit message: Updated with the last values of Stephane

File: urdfs/sensors/bumblebee.urdf.xacro (robot description, xacro)
@@ -13,10 +13,9 @@
 			<parent link="${frame_prefix}mount_link"/>
 			<child link="${frame_prefix}optical_frame"/>
-			<!--<origin xyz="0 0 0" rpy="0 0 0"/>-->
-			<origin xyz="0 -0.06 0" rpy="-${PI/2} 0 -${PI/2}"/>
+			<origin xyz="0 -0.06 0.018" rpy="-${PI/2} 0 -${PI/2}"/>
 		</joint>
 		<link name="${frame_prefix}mount_link">
 			<visual>
-				<origin xyz="0 0 0" rpy="${PI/2} 0 ${PI/2}"/>
+				<origin xyz="0 0 0.018" rpy="${PI/2} 0 ${PI/2}"/>
 				<geometry>
 					<mesh filename="package://hyq2max_description/meshes/sensors/bumblebee.dae"/>
@@ -24,5 +23,5 @@
 			</visual>
 			<collision>
-				<origin xyz="0 0 0" rpy="${PI/2} 0 ${PI/2}"/>
+				<origin xyz="0 0 0.018" rpy="${PI/2} 0 ${PI/2}"/>
 				<geometry>
 					<mesh filename="package://hyq2max_description/meshes/sensors/bumblebee.dae"/>
@@ -34,5 +33,5 @@
 						 iyy="${1/12*b2mass*(b2lx*b2lx + b2lz*b2lz)}" iyz="0"
 						 izz="${1/12*b2mass*(b2lx*b2lx + b2ly*b2ly)}" />
-				</inertial>
+			</inertial>
 		</link>
 		<link name="${frame_prefix}optical_frame">

File: urdfs/sensors/ptu_d46.urdf.xacro (robot description, xacro)
@@ -64,5 +64,5 @@
         	 the overall device, which is between the mounting screws on its base. -->
 		<joint name="${name}_base" type="fixed">
-			<origin xyz="0 -0.011 0.022" rpy="0 0 0"/>
+			<origin xyz="0 -0.0127254 0.022" rpy="0 0 0"/>
 			<parent link="${name}_base_link"/>
 			<child link="${name}_pan_link"/>
@@ -78,5 +78,5 @@
 		<!-- The tilt joint -->
 		<joint name="${name}_tilt" type="revolute">
-			<origin xyz="0 0 0" rpy="-${PI/2} 0 0"/>
+			<origin xyz="0 -0.002424 0" rpy="-${PI/2} 0 0"/>
 			<parent link="${name}_tilt_link"/>
 			<child link="${name}_tilted_link"/>
@@ -86,5 +86,5 @@
 		<!-- Fixed joint to provide a convenient attachment point for accessories. -->
 		<joint name="${name}_mount" type="fixed">
-			<origin xyz="0 0 -0.03912" rpy="${PI} 0 0"/>
+			<origin xyz="0 0 -0.039116" rpy="${PI} 0 0"/>
 			<parent link="${name}_tilted_link"/>
 			<child link="${name}_mount_link"/>
