Commit message: [bugfix] Fixed the joint limits (Felipe and Victor)

File: urdfs/leg/leg.urdf.xacro (robot description, xacro)
@@ -33,5 +33,5 @@
 		<!-- Lower leg joint -->
 		<joint name="${name}_kfe_joint" type="revolute">
-			<origin xyz="${lowerleg_length} 0 0" rpy="0 0 0"/>
+			<origin xyz="${lowerleg_length} 0 0" rpy="0 0 ${-reflect_front*9.8*PI/180}"/>
 			<parent link="${name}_upperleg"/>
 			<child  link="${name}_lowerleg"/>
@@ -39,9 +39,9 @@
 			<dynamics damping="0.1" friction="0" />
 			<limit effort="150.0" velocity="12.0"
-				   lower="${(1-reflect_front)*3*PI/360-(1+reflect_front)*163*PI/360}"
-				   upper="${(1-reflect_front)*163*PI/360-(1+reflect_front)*3*PI/360}"/>
+				   lower="${-(1+reflect_front)*167*PI/360}"
+				   upper="${(1-reflect_front)*167*PI/360}"/>
 			<safety_controller k_position="100" k_velocity="100"
-							   soft_lower_limit="${(1-reflect_front)*3*PI/360-(1+reflect_front)*163*PI/360}"
-							   soft_upper_limit="${(1-reflect_front)*163*PI/360-(1+reflect_front)*3*PI/360}" />
+							   soft_lower_limit="${-(1+reflect_front)*167*PI/360}"
+							   soft_upper_limit="${(1-reflect_front)*167*PI/360}" />
 		</joint>
 		<!-- Foot joint -->

Commit message: Corrected the Leg Joint Torques, ready to make the repository public

File: urdfs/leg/leg.urdf.xacro (robot description, xacro)
@@ -15,5 +15,5 @@
 			<axis xyz="0 0 1"/>
 			<dynamics damping="0.1" friction="0" />
-			<limit effort="150.0" velocity="12.0" lower="${-2*PI/9}" upper="${2*PI/9}"/>
+			<limit effort="120.0" velocity="12.0" lower="${-2*PI/9}" upper="${2*PI/9}"/>
 			<safety_controller k_position="100" k_velocity="100"
 							   soft_lower_limit="${-2*PI/9}" soft_upper_limit="${2*PI/9}" />
@@ -27,5 +27,5 @@
 			<axis xyz="0 0 1"/>
 			<dynamics damping="0.1" friction="0" />
-			<limit effort="150.0" velocity="12.0" lower="${-3*PI/4}" upper="${3*PI/4}"/>
+			<limit effort="245.0" velocity="12.0" lower="${-3*PI/4}" upper="${3*PI/4}"/>
 			<safety_controller k_position="100" k_velocity="100"
 							   soft_lower_limit="${-3*PI/4}" soft_upper_limit="${3*PI/4}" />
@@ -38,5 +38,5 @@
 			<axis xyz="0 0 1"/>
 			<dynamics damping="0.1" friction="0" />
-			<limit effort="150.0" velocity="12.0"
+			<limit effort="250.0" velocity="12.0"
 				   lower="${-(1+reflect_front)*167*PI/360}"
 				   upper="${(1-reflect_front)*167*PI/360}"/>

Commit message: [config] Removed the mass of the foot

File: urdfs/leg/leg.urdf.xacro (robot description, xacro)
@@ -120,5 +120,5 @@
 			<inertial>
 				<origin xyz="0 0 0"/>
-				<mass value="0.01"/>
+				<mass value="0.0"/>
 				<inertia ixx="0.0" iyy="0.0" izz="0.0" ixy="0.0" ixz="0.0" iyz="0.0"/>
 			</inertial>

Commit message: [cleanup] Removed comment lines after checking them

File: urdfs/leg/leg.urdf.xacro (robot description, xacro)
@@ -61,5 +61,5 @@
 			</inertial>
 			<visual>
-				<origin xyz="0 -0.046 0" rpy="0 ${-PI/2} ${-PI/2}"/><!-- TODO: -0.044 ask Jake -->
+				<origin xyz="0 -0.046 0" rpy="0 ${-PI/2} ${-PI/2}"/>
 				<geometry>
 					<mesh filename="package://hyq2max_description/meshes/leg/hipassembly.dae" scale="1 1 1"/>
@@ -67,5 +67,5 @@
 			</visual>
 			<collision>
-				<origin xyz="0 -0.046 0" rpy="0 ${-PI/2} ${-PI/2}"/><!-- TODO: -0.044 ask Jake -->
+				<origin xyz="0 -0.046 0" rpy="0 ${-PI/2} ${-PI/2}"/>
 				<geometry>
 					<mesh filename="package://hyq2max_description/meshes/leg/hipassembly.dae" scale="1 1 1"/>
@@ -82,5 +82,5 @@
 			</inertial>
 			<visual>
-				<origin xyz="0 0 ${-0.03*reflect_left}" rpy="${(1-reflect_left)*PI/2} 0 0"/> <!-- TODO Ask displacement Jake -->
+				<origin xyz="0 0 ${-0.03*reflect_left}" rpy="${(1-reflect_left)*PI/2} 0 0"/>
 				<geometry>
 					<mesh filename="package://hyq2max_description/meshes/leg/upperleg.dae" scale="1 1 1"/>
@@ -88,5 +88,5 @@
 			</visual>
 			<collision>
-				<origin xyz="0 0 ${-0.03*reflect_left}" rpy="${(1-reflect_left)*PI/2} 0 0"/> <!-- TODO Ask displacement Jake -->
+				<origin xyz="0 0 ${-0.03*reflect_left}" rpy="${(1-reflect_left)*PI/2} 0 0"/>
 				<geometry>
 					<mesh filename="package://hyq2max_description/meshes/leg/upperleg.dae" scale="1 1 1"/>

Commit message: corrected kin limits according to Alex email

File: urdfs/leg/leg.urdf.xacro (robot description, xacro)
@@ -38,10 +38,10 @@
 			<axis xyz="0 0 1"/>
 			<dynamics damping="0.1" friction="0" />
-			<limit effort="250.0" velocity="12.0"
-				   lower="${(1-reflect_front)*2*PI/360-(1+reflect_front)*167*PI/360}"
-				   upper="${-(1+reflect_front)*2*PI/360+(1-reflect_front)*167*PI/360}"/>
-			<safety_controller k_position="100" k_velocity="100"
-							   soft_lower_limit="${-(1+reflect_front)*167*PI/360}"
-							   soft_upper_limit="${(1-reflect_front)*167*PI/360}" />
+            <limit effort="250.0" velocity="12.0"
+                   lower="${(1-reflect_front)*2*PI/180-(1+reflect_front)*167*PI/180}"
+                   upper="${-(1+reflect_front)*2*PI/180+(1-reflect_front)*167*PI/180}"/>
+            <safety_controller k_position="100" k_velocity="100"
+                               soft_lower_limit="${(1-reflect_front)*2*PI/180-(1+reflect_front)*167*PI/180}"
+                               soft_upper_limit="${-(1+reflect_front)*2*PI/180+(1-reflect_front)*167*PI/180}" />
 		</joint>
 		<!-- Foot joint -->
