Commit message: Added the upperleg and foot collision information

File: urdfs/leg/leg.gazebo.xacro (robot description, xacro)
@@ -2,4 +2,13 @@
 <robot xmlns:xacro="http://www.ros.org/wiki/xacro">
 	<xacro:macro name="leg_gazebo" params="name">
+		<gazebo reference="${name}_upperleg">
+			<kp>1000000.0</kp>
+			<kd>100.0</kd>
+			<mu1>1.5</mu1>
+			<mu2>1.5</mu2>
+			<fdir1>1 0 0</fdir1>
+			<maxVel>1.0</maxVel>
+			<minDepth>0.00</minDepth>
+		</gazebo>
 		<gazebo reference="${name}_lowerleg">
 			<kp>1000000.0</kp>
@@ -11,4 +20,15 @@
 			<minDepth>0.00</minDepth>
 		</gazebo>
+		<gazebo reference="${name}_foot">
+			<!-- contact sensor -->
+			<sensor type="contact" name="${name}_foot_contact_sensor">
+				<update_rate>1000.0</update_rate>
+				<always_on>1</always_on>
+				<contact>
+					<collision>${name}_foot_collision</collision>
+					<topic>/${name}_foot_contact</topic>
+				</contact>
+			</sensor>
+		</gazebo>
 	</xacro:macro>
 </robot>

Commit message: added shin collision sensor

File: urdfs/leg/leg.gazebo.xacro (robot description, xacro)
@@ -50,13 +50,23 @@
 			<minDepth>0.00</minDepth>
 		</gazebo>
-		<gazebo reference="${name}_lowerleg">
-			<kp>1000000.0</kp>
-			<kd>100.0</kd>
-			<mu1>1.5</mu1>
-			<mu2>1.5</mu2>
-			<fdir1>1 0 0</fdir1>
-			<maxVel>1.0</maxVel>
-			<minDepth>0.00</minDepth>
-		</gazebo>
+    	 <gazebo reference="${name}_lowerleg">
+            <kp>1000000.0</kp>
+            <kd>100.0</kd>
+            <mu1>1.5</mu1>
+            <mu2>1.5</mu2>
+            <fdir1>1 0 0</fdir1>
+            <maxVel>1.0</maxVel>
+            <minDepth>0.00</minDepth>
+            <sensor name="${name}_shin_contact_sensor" type="contact">
+                <always_on>true</always_on>
+                <update_rate>1000.0</update_rate>
+                <contact>
+                  <collision>${name}_lowerleg_collision</collision>
+                </contact>
+                <plugin name="${name}_shin_bumper" filename="libgazebo_ros_bumper.so">
+                  <bumperTopicName>/${name}_shin_sensor</bumperTopicName>
+                </plugin>
+            </sensor>
+        </gazebo>
 		<gazebo reference="${name}_foot">
 			<sensor name="${name}_foot_contact_sensor" type="contact">
