Commit message: [bugfix] Defined a proper orientation of the knee reference system

File: urdfs/common.xacro (robot description, xacro)
@@ -7,4 +7,6 @@
 	<property name="upperleg_length" value="0.1075"/>
 	<property name="lowerleg_length" value="0.364"/>
+	<!-- Knee offset angel in degree -->
+	<property name="knee_offset_angle" value="10"/>
 	<!-- Inertial values -->
 	<!-- Trunk with hydraulic system -->

File: urdfs/leg/leg.urdf.xacro (robot description, xacro)
@@ -33,5 +33,5 @@
 		<!-- Lower leg joint -->
 		<joint name="${name}_kfe_joint" type="revolute">
-			<origin xyz="${lowerleg_length} 0 0" rpy="0 0 ${-reflect_front*9.8*PI/180}"/>
+			<origin xyz="${lowerleg_length} 0 0" rpy="0 0 ${reflect_front*knee_offset_angle*PI/180}"/>
 			<parent link="${name}_upperleg"/>
 			<child  link="${name}_lowerleg"/>
@@ -39,6 +39,6 @@
 			<dynamics damping="0.1" friction="0" />
 			<limit effort="250.0" velocity="12.0"
-				   lower="${-(1+reflect_front)*167*PI/360}"
-				   upper="${(1-reflect_front)*167*PI/360}"/>
+				   lower="${(1-reflect_front)*2*PI/360-(1+reflect_front)*167*PI/360}"
+				   upper="${-(1+reflect_front)*2*PI/360+(1-reflect_front)*167*PI/360}"/>
 			<safety_controller k_position="100" k_velocity="100"
 							   soft_lower_limit="${-(1+reflect_front)*167*PI/360}"
@@ -47,5 +47,5 @@
 		<!-- Foot joint -->
 		<joint name="${name}_foot_joint" type="fixed">
-			<origin xyz="0.37432 ${reflect_front*0.066} 0" rpy="${PI/2} 0 ${-PI/2}"/>
+			<origin xyz="0.380094 0 0" rpy="${PI/2} 0 ${-PI/2}"/>
 			<parent link="${name}_lowerleg"/>
 			<child  link="${name}_foot"/>
@@ -103,5 +103,5 @@
 			</inertial>
 			<visual>
-				<origin xyz="0 0 0" rpy="${(1-reflect_front)*PI/2} 0 ${PI}"/> <!-- TODO Ask displacement Jake -->
+				<origin xyz="0 0 0" rpy="${(1-reflect_front)*PI/2} 0 ${PI-reflect_front*knee_offset_angle*PI/180}"/>
 				<geometry>
 					<mesh filename="package://hyq2max_description/meshes/leg/lowerleg.dae" scale="1 1 1"/>
@@ -110,5 +110,5 @@
 			</visual>
 			<collision>
-				<origin xyz="0 0 0" rpy="${(1-reflect_front)*PI/2} 0 ${PI}"/> <!-- TODO Ask displacement Jake -->
+				<origin xyz="0 0 0" rpy="${(1-reflect_front)*PI/2} 0 ${PI-reflect_front*knee_offset_angle*PI/180}"/>
 				<geometry>
 					<mesh filename="package://hyq2max_description/meshes/leg/lowerleg.dae" scale="1 1 1"/>

Commit message: renamed some variables
added lowerleg length variable

File: urdfs/common.xacro (robot description, xacro)
@@ -5,6 +5,7 @@
 	<property name="d_lr" value="0.414"/>
 	<property name="d_fh" value="0.747"/>
-	<property name="upperleg_length" value="0.1075"/>
-	<property name="lowerleg_length" value="0.364"/>
+	<property name="hipassembly_length" value="0.1075"/>
+	<property name="upperleg_length" value="0.364"/>
+    <property name="lowerleg_length" value="0.38009"/>
 	<!-- Inertial values -->
 	<!-- Trunk with hydraulic system -->

File: urdfs/leg/leg.urdf.xacro (robot description, xacro)
@@ -8,5 +8,5 @@
 	<xacro:macro name="hyq2max_leg" params="name parent *origin reflect_left reflect_front">
 		<!-- Joints -->
-		<!-- Hip assembly joint -->
+		<!-- HAA joint -->
 		<joint name="${name}_haa_joint" type="revolute">
 			<insert_block name="origin"/>
@@ -19,7 +19,7 @@
 							   soft_lower_limit="${-2*PI/9}" soft_upper_limit="${2*PI/9}" />
 		</joint>
-		<!-- Upper leg joint -->
+		<!-- HFE joint -->
 		<joint name="${name}_hfe_joint" type="revolute">
-			<origin xyz="0 ${-upperleg_length} 0"
+			<origin xyz="0 ${-hipassembly_length} 0"
 					rpy="${reflect_left*PI/2} 0 0"/>
 			<parent link="${name}_hipassembly"/>
@@ -31,7 +31,7 @@
 							   soft_lower_limit="${-3*PI/4}" soft_upper_limit="${3*PI/4}" />
 		</joint>
-		<!-- Lower leg joint -->
+		<!-- KFE joint -->
 		<joint name="${name}_kfe_joint" type="revolute">
-			<origin xyz="${lowerleg_length} 0 0" rpy="0 0 ${-reflect_front*9.8*PI/180}"/>
+			<origin xyz="${upperleg_length} 0 0" rpy="0 0 ${-reflect_front*9.8*PI/180}"/>
 			<parent link="${name}_upperleg"/>
 			<child  link="${name}_lowerleg"/>
@@ -47,5 +47,5 @@
 		<!-- Foot joint -->
 		<joint name="${name}_foot_joint" type="fixed">
-			<origin xyz="0.37432 ${reflect_front*0.066} 0" rpy="${PI/2} 0 ${-PI/2}"/>
+			<origin xyz="${lowerleg_length} 0 0" rpy="${PI/2} 0 ${-PI/2}"/>
 			<parent link="${name}_lowerleg"/>
 			<child  link="${name}_foot"/>

Commit message: [bugfix] Removed the offset in the knee joints

File: urdfs/common.xacro (robot description, xacro)
@@ -9,5 +9,5 @@
     <property name="lowerleg_length" value="0.38009"/>
 	<!-- Knee offset angel in degree -->
-	<property name="knee_offset_angle" value="10"/>
+	<property name="knee_offset_angle" value="10."/>
 	<!-- Inertial values -->
 	<!-- Trunk with hydraulic system -->

File: urdfs/leg/leg.urdf.xacro (robot description, xacro)
@@ -33,5 +33,5 @@
 		<!-- KFE joint -->
 		<joint name="${name}_kfe_joint" type="revolute">
-			<origin xyz="${upperleg_length} 0 0" rpy="0 0 ${reflect_front*knee_offset_angle*PI/180}"/>
+			<origin xyz="${upperleg_length} 0 0" rpy="0 0 0"/>
 			<parent link="${name}_upperleg"/>
 			<child  link="${name}_lowerleg"/>

Commit message: parameterised values, renewed meshes and tuned launch file

File: urdfs/common.xacro (robot description, xacro)
@@ -5,4 +5,10 @@
 	<property name="d_lr" value="0.414"/>
 	<property name="d_fh" value="0.747"/>
+	<property name="haa_lr" value="0.194"/>
+	<!-- 0.194  0.34125 -->
+	<property name="haa_fh" value="0.887"/>
+	<!-- 0.887 1.4192-->
+	<property name="trunkScale_width" value="${haa_lr/0.194}"/>
+	<property name="trunkScale_length" value="${haa_fh/0.887}"/>
 	<property name="hipassembly_length" value="0.117"/>
 	<property name="upperleg_length" value="0.360"/>

File: urdfs/leg/leg.urdf.xacro (robot description, xacro)
@@ -63,14 +63,19 @@
 				<origin xyz="0 -0.046 0" rpy="0 ${-PI/2} ${-PI/2}"/>
 				<geometry>
-					<mesh filename="package://hyq2max_description/meshes/leg/hipassembly.dae" scale="1 1 1"/>
+				<cylinder length="0.117" radius="0.0444"/>
 				</geometry>
+                                <material name="black"/>
 			</visual>
 			<collision>
 				<origin xyz="0 -0.046 0" rpy="0 ${-PI/2} ${-PI/2}"/>
 				<geometry>
-					<mesh filename="package://hyq2max_description/meshes/leg/hipassembly.dae" scale="1 1 1"/>
+					<!-- <mesh filename="package://hyq2max_description/meshes/leg/hipassembly.dae" scale="1 1 1"/> -->
+				<cylinder length="0.117" radius="0.0444"/>
 				</geometry>
 			</collision>
 		</link>
+		<gazebo reference="${name}_hipassembly">
+            		<material>Gazebo/Black</material>
+	        </gazebo>
 		<!-- Upper leg link -->
 		<link name="${name}_upperleg">
@@ -83,12 +88,18 @@
 			<visual>
 				<origin xyz="0 0 ${-0.03*reflect_left}" rpy="${(1-reflect_left)*PI/2} 0 0"/>
+				<!-- <origin xyz="0.180 0 0" rpy="0 0 0"/> -->
 				<geometry>
 					<mesh filename="package://hyq2max_description/meshes/leg/upperleg.dae" scale="1 1 1"/>
+				<!-- <box size="0.360 0.116 0.07"/> -->
+				<!-- <cylinder length="0.360" radius="0.07"/> -->
 				</geometry>
 			</visual>
 			<collision>
 				<origin xyz="0 0 ${-0.03*reflect_left}" rpy="${(1-reflect_left)*PI/2} 0 0"/>
+				<!-- <origin xyz="0.180 0 0" rpy="0 0 0"/> -->
 				<geometry>
 					<mesh filename="package://hyq2max_description/meshes/leg/upperleg.dae" scale="1 1 1"/>
+				<!-- <box size="0.360 0.116 0.07"/> -->
+				<!-- <cylinder length="0.360" radius="0.07"/> -->
 				</geometry>
 			</collision>
@@ -123,10 +134,11 @@
 				<inertia ixx="0.0" iyy="0.0" izz="0.0" ixy="0.0" ixz="0.0" iyz="0.0"/>
 			</inertial>
-			<!--<visual>
+			<visual>
 				<origin xyz="0.0 0.0 0.0" rpy="0.0 0.0 0.0"/>
 				<geometry>
 					<sphere radius="0.021"/>
 				</geometry>
-			</visual>-->
+                                <material name="black"/>
+			</visual>
 			<collision>
 				<origin xyz="0 0 0" rpy="0 0 0"/>
@@ -136,4 +148,7 @@
 			</collision>
 		</link>
+                <gazebo reference="${name}_foot">
+                	<material>Gazebo/Black</material>
+                </gazebo>
 		<!-- Extensions -->
 		<xacro:leg_transmission name="${name}"/>

File: urdfs/trunk/trunk.urdf.xacro (robot description, xacro)
@@ -31,12 +31,16 @@
 			<visual>
 				<origin xyz="0 0 0" rpy="${PI/2} 0 ${PI/2}" />
+				<!-- <origin xyz="0 0 0" rpy="0 0 0" /> -->
 				<geometry>
-					<mesh filename="package://hyq2max_description/meshes/trunk/trunk.dae" scale="1 1 1"/>
+ 					<mesh filename="package://hyq2max_description/meshes/trunk/trunk.dae" scale="${trunkScale_width} 1 ${trunkScale_length}"/>
+				 <!-- <box size="1.306 0.400 0.318"/>  -->
 				</geometry>
 			</visual>
 			<collision>
 				<origin xyz="0 0 0" rpy="${PI/2} 0 ${PI/2}" />
+				<!-- <origin xyz="0 0 0" rpy="0 0 0" /> -->
 				<geometry>
-					<mesh filename="package://hyq2max_description/meshes/trunk/trunk.dae" scale="1 1 1"/>
+					<mesh filename="package://hyq2max_description/meshes/trunk/trunk.dae" scale="${trunkScale_width} 1 ${trunkScale_length}"/>
+				<!-- <box size="1.306 0.400 0.318"/>  -->
 				</geometry>
 			</collision>

Commit message: default hyq2max values. parameterised trunk dimensions

File: urdfs/common.xacro (robot description, xacro)
@@ -9,4 +9,6 @@
 	<property name="haa_fh" value="0.887"/>
 	<!-- 0.887 1.4192-->
+	<property name="trunkScale_width" value="${haa_lr/0.194}"/>
+	<property name="trunkScale_length" value="${haa_fh/0.887}"/>
 	<property name="hipassembly_length" value="0.117"/>
 	<property name="upperleg_length" value="0.360"/>
@@ -19,11 +21,11 @@
 	<property name="ycom_trunk" value="0.000598"/>
 	<property name="zcom_trunk" value="-0.007592"/>
-	<property name="m_trunk" value="79.71"/>
-	<property name="ixx_trunk" value="0.606365070385293"/>
-	<property name="iyy_trunk" value="9.537595569881642"/>
-	<property name="izz_trunk" value="9.683530508687989"/>
-	<property name="ixy_trunk" value="-0.010207938403425"/>
-	<property name="ixz_trunk" value="0.009349214202972"/>
-	<property name="iyz_trunk" value="-0.003535462679426"/>
+	<property name="m_trunk" value="39.71"/>
+	<property name="ixx_trunk" value="0.3020795"/>
+	<property name="iyy_trunk" value="4.751448"/>
+	<property name="izz_trunk" value="4.82415"/>
+	<property name="ixy_trunk" value="-0.0050854"/>
+	<property name="ixz_trunk" value=" 0.0046576"/>
+	<property name="iyz_trunk" value="-0.0017613"/>
 	<!-- Hip assembly -->
 	<property name="xcom_hipassembly" value="-0.000605"/>

File: urdfs/trunk/trunk.urdf.xacro (robot description, xacro)
@@ -32,5 +32,5 @@
 				<origin xyz="0 0 0" rpy="${PI/2} 0 ${PI/2}" />
 				<geometry>
-					<mesh filename="package://hyq2max_description/meshes/trunk/trunk.dae" scale="1 1 1"/>
+					<mesh filename="package://hyq2max_description/meshes/trunk/trunk.dae" scale="${trunkScale_width} 1 ${trunkScale_length}"/>
 				</geometry>
 			</visual>
@@ -38,5 +38,5 @@
 				<origin xyz="0 0 0" rpy="${PI/2} 0 ${PI/2}" />
 				<geometry>
-					<mesh filename="package://hyq2max_description/meshes/trunk/trunk.dae" scale="1 1 1"/>
+					<mesh filename="package://hyq2max_description/meshes/trunk/trunk.dae" scale="${trunkScale_width} 1 ${trunkScale_length}"/>
 				</geometry>
 			</collision>

File: urdfs/trunk/trunk_model.urdf.xacro (robot description, xacro)
@@ -32,5 +32,5 @@
 				<origin xyz="0 0 0" rpy="${PI/2} 0 ${PI/2}" />
 				<geometry>
-					<mesh filename="package://hyq2max_description/meshes/trunk/trunk.dae" scale="1 1 1"/>
+					<mesh filename="package://hyq2max_description/meshes/trunk/trunk.dae" scale="${trunkScale_width} 1 ${trunkScale_length}"/>
 				</geometry>
 			</visual>
@@ -38,5 +38,5 @@
 				<origin xyz="0 0 0" rpy="${PI/2} 0 ${PI/2}" />
 				<geometry>
-					<mesh filename="package://hyq2max_description/meshes/trunk/trunk.dae" scale="1 1 1"/>
+					<mesh filename="package://hyq2max_description/meshes/trunk/trunk.dae" scale="${trunkScale_width} 1 ${trunkScale_length}"/>
 				</geometry>
 			</collision>

Commit message: Fix in xacro tags (warnings)

File: urdfs/common.xacro (robot description, xacro)
@@ -1,63 +1,63 @@
 <?xml version="1.0"?>
 <robot>
-	<property name="PI" value="3.1415926535897931"/>
+	<xacro:property name="PI" value="3.1415926535897931"/>
 	<!-- standard distances -->
-	<property name="d_lr" value="0.414"/>
-	<property name="d_fh" value="0.747"/>
-	<property name="haa_lr" value="0.194"/>
+	<xacro:property name="d_lr" value="0.414"/>
+	<xacro:property name="d_fh" value="0.747"/>
+	<xacro:property name="haa_lr" value="0.194"/>
 	<!-- 0.194  0.34125 -->
-	<property name="haa_fh" value="0.887"/>
+	<xacro:property name="haa_fh" value="0.887"/>
 	<!-- 0.887 1.4192-->
-	<property name="trunkScale_width" value="${haa_lr/0.194}"/>
-	<property name="trunkScale_length" value="${haa_fh/0.887}"/>
-	<property name="hipassembly_length" value="0.117"/>
-	<property name="upperleg_length" value="0.360"/>
-    <property name="lowerleg_length" value="0.380"/>
+	<xacro:property name="trunkScale_width" value="${haa_lr/0.194}"/>
+	<xacro:property name="trunkScale_length" value="${haa_fh/0.887}"/>
+	<xacro:property name="hipassembly_length" value="0.117"/>
+	<xacro:property name="upperleg_length" value="0.360"/>
+    <xacro:property name="lowerleg_length" value="0.380"/>
 	<!-- Knee offset angel in degree -->
-	<property name="knee_offset_angle" value="10."/>
+	<xacro:property name="knee_offset_angle" value="10."/>
 	<!-- Inertial values -->
 	<!-- Trunk with hydraulic system -->
-	<property name="xcom_trunk" value="0.060663"/>
-	<property name="ycom_trunk" value="0.000598"/>
-	<property name="zcom_trunk" value="-0.007592"/>
-	<property name="m_trunk" value="39.71"/>
-	<property name="ixx_trunk" value="0.3020795"/>
-	<property name="iyy_trunk" value="4.751448"/>
-	<property name="izz_trunk" value="4.82415"/>
-	<property name="ixy_trunk" value="-0.0050854"/>
-	<property name="ixz_trunk" value="0.0046576"/>
-	<property name="iyz_trunk" value="-0.0017613"/>
+	<xacro:property name="xcom_trunk" value="0.060663"/>
+	<xacro:property name="ycom_trunk" value="0.000598"/>
+	<xacro:property name="zcom_trunk" value="-0.007592"/>
+	<xacro:property name="m_trunk" value="39.71"/>
+	<xacro:property name="ixx_trunk" value="0.3020795"/>
+	<xacro:property name="iyy_trunk" value="4.751448"/>
+	<xacro:property name="izz_trunk" value="4.82415"/>
+	<xacro:property name="ixy_trunk" value="-0.0050854"/>
+	<xacro:property name="ixz_trunk" value="0.0046576"/>
+	<xacro:property name="iyz_trunk" value="-0.0017613"/>
 	<!-- Hip assembly -->
-	<property name="xcom_hipassembly" value="-0.000605"/>
-	<property name="ycom_hipassembly" value="-0.001346"/>
-	<property name="zcom_hipassembly" value="0.000196"/>
-	<property name="m_hipassembly" value="3.54"/>
-	<property name="ixx_hipassembly" value="0.007379"/>
-	<property name="iyy_hipassembly" value="0.004284"/>
-	<property name="izz_hipassembly" value="0.007090"/>
-	<property name="ixy_hipassembly" value="-0.000053"/>
-	<property name="ixz_hipassembly" value="0.000017"/>
-	<property name="iyz_hipassembly" value="0.000030"/>
+	<xacro:property name="xcom_hipassembly" value="-0.000605"/>
+	<xacro:property name="ycom_hipassembly" value="-0.001346"/>
+	<xacro:property name="zcom_hipassembly" value="0.000196"/>
+	<xacro:property name="m_hipassembly" value="3.54"/>
+	<xacro:property name="ixx_hipassembly" value="0.007379"/>
+	<xacro:property name="iyy_hipassembly" value="0.004284"/>
+	<xacro:property name="izz_hipassembly" value="0.007090"/>
+	<xacro:property name="ixy_hipassembly" value="-0.000053"/>
+	<xacro:property name="ixz_hipassembly" value="0.000017"/>
+	<xacro:property name="iyz_hipassembly" value="0.000030"/>
 	<!-- Upper leg -->
-	<property name="xcom_upperleg" value="0.144296"/>
-	<property name="ycom_upperleg" value="-0.002071"/>
-	<property name="zcom_upperleg" value="-0.005094"/>
-	<property name="m_upperleg" value="4.95"/>
-	<property name="ixx_upperleg" value="0.010196"/>
-	<property name="iyy_upperleg" value="0.204183"/>
-	<property name="izz_upperleg" value="0.207532"/>
-	<property name="ixy_upperleg" value="-0.002320"/>
-	<property name="ixz_upperleg" value="-0.000141"/>
-	<property name="iyz_upperleg" value="0.000034"/>
+	<xacro:property name="xcom_upperleg" value="0.144296"/>
+	<xacro:property name="ycom_upperleg" value="-0.002071"/>
+	<xacro:property name="zcom_upperleg" value="-0.005094"/>
+	<xacro:property name="m_upperleg" value="4.95"/>
+	<xacro:property name="ixx_upperleg" value="0.010196"/>
+	<xacro:property name="iyy_upperleg" value="0.204183"/>
+	<xacro:property name="izz_upperleg" value="0.207532"/>
+	<xacro:property name="ixy_upperleg" value="-0.002320"/>
+	<xacro:property name="ixz_upperleg" value="-0.000141"/>
+	<xacro:property name="iyz_upperleg" value="0.000034"/>
 	<!-- Lower leg -->
-	<property name="xcom_lowerleg" value="0.109015"/>
-	<property name="ycom_lowerleg" value="0.042147"/>
-	<property name="zcom_lowerleg" value="0.000219"/>
-	<property name="m_lowerleg" value="1.71"/>
-	<property name="ixx_lowerleg" value="0.006848"/>
-	<property name="iyy_lowerleg" value="0.055957"/>
-	<property name="izz_lowerleg" value="0.059397"/>
-	<property name="ixy_lowerleg" value="0.011981"/>
-	<property name="ixz_lowerleg" value="0.000008"/>
-	<property name="iyz_lowerleg" value="0.000012"/>
+	<xacro:property name="xcom_lowerleg" value="0.109015"/>
+	<xacro:property name="ycom_lowerleg" value="0.042147"/>
+	<xacro:property name="zcom_lowerleg" value="0.000219"/>
+	<xacro:property name="m_lowerleg" value="1.71"/>
+	<xacro:property name="ixx_lowerleg" value="0.006848"/>
+	<xacro:property name="iyy_lowerleg" value="0.055957"/>
+	<xacro:property name="izz_lowerleg" value="0.059397"/>
+	<xacro:property name="ixy_lowerleg" value="0.011981"/>
+	<xacro:property name="ixz_lowerleg" value="0.000008"/>
+	<xacro:property name="iyz_lowerleg" value="0.000012"/>
 </robot>

File: urdfs/leg/leg.urdf.xacro (robot description, xacro)
@@ -10,5 +10,5 @@
 		<!-- HAA joint -->
 		<joint name="${name}_haa_joint" type="revolute">
-			<insert_block name="origin"/>
+			<xacro:insert_block name="origin"/>
 			<parent link="${parent}"/>
 			<child  link="${name}_hipassembly"/>
