Commit message: Changed sensor path to the correct path

File: robots/hyq2max.urdf.xacro (robot description, xacro)
@@ -1,4 +1,4 @@
 <?xml version="1.0"?>
-<robot name="hyq" xmlns:xacro="http://www.ros.org/wiki/xacro">
+<robot name="hyq2max" xmlns:xacro="http://www.ros.org/wiki/xacro">
 	<!-- The following included files set up definitions of parts of the robot body -->
 	<xacro:include filename="$(find hyq2max_description)/urdfs/common.xacro"/>

File: urdfs/sensors/asus_xtion.urdf.xacro (robot description, xacro)
@@ -45,5 +45,5 @@
 				<origin xyz="0 0 0" rpy="0 0 0"/>
 				<geometry>
-					<mesh filename="package://hyq_description/meshes/sensors/asus_xtion.dae" scale="1 1 1" />
+					<mesh filename="package://hyq2max_description/meshes/sensors/asus_xtion.dae" scale="1 1 1" />
 				</geometry>
 				<material name="gray">

File: urdfs/sensors/bumblebee.urdf.xacro (robot description, xacro)
@@ -20,5 +20,5 @@
 				<origin xyz="0 0 0" rpy="${PI/2} 0 ${PI/2}"/>
 				<geometry>
-					<mesh filename="package://hyq_description/meshes/sensors/bumblebee.dae"/>
+					<mesh filename="package://hyq2max_description/meshes/sensors/bumblebee.dae"/>
 				</geometry>
 			</visual>
@@ -26,5 +26,5 @@
 				<origin xyz="0 0 0" rpy="${PI/2} 0 ${PI/2}"/>
 				<geometry>
-					<mesh filename="package://hyq_description/meshes/sensors/bumblebee.dae"/>
+					<mesh filename="package://hyq2max_description/meshes/sensors/bumblebee.dae"/>
 				</geometry>
 			</collision>

File: urdfs/sensors/kinect.urdf.xacro (robot description, xacro)
@@ -46,5 +46,5 @@
 				<origin xyz="0.0 0.0 0.0" rpy="0.0 0.0 0"/>
 				<geometry>
-					<mesh filename="package://hyq_description/meshes/sensors/kinect.dae" scale="1 1 1" />
+					<mesh filename="package://hyq2max_description/meshes/sensors/kinect.dae" scale="1 1 1" />
 				</geometry>
 				<material name="gray">
@@ -55,5 +55,5 @@
 				<origin xyz="0.0 0.0 0.0" rpy="0.0 0.0 0.0"/>
 				<geometry>
-					<mesh filename="package://hyq_description/meshes/sensors/kinect.dae" scale="1 1 1" />
+					<mesh filename="package://hyq2max_description/meshes/sensors/kinect.dae" scale="1 1 1" />
 				</geometry>
 			</collision>

File: urdfs/sensors/velodyne.urdf.xacro (robot description, xacro)
@@ -27,5 +27,5 @@
 				<origin xyz="0 0 0" rpy="0 0 0"/>
 				<geometry>
-					<mesh filename="package://hyq_description/meshes/sensors/velodyne_hdl32e.dae" scale="1 1 1" />
+					<mesh filename="package://hyq2max_description/meshes/sensors/velodyne_hdl32e.dae" scale="1 1 1" />
 				</geometry>
 				<material name="gray">

File: urdfs/sensors/vislab_3dve.urdf.xacro (robot description, xacro)
@@ -18,5 +18,5 @@
 				<origin xyz="0.018 0 0" rpy="${PI/2} 0 ${-PI/2}"/>
 				<geometry>
-					<mesh filename="package://hyq_description/meshes/sensors/vislab_3dve.stl"/>
+					<mesh filename="package://hyq2max_description/meshes/sensors/vislab_3dve.stl"/>
 				</geometry>
 			</visual>
@@ -24,5 +24,5 @@
 				<origin xyz="0.018 0 0" rpy="${PI/2} 0 ${-PI/2}"/>
 				<geometry>
-					<mesh filename="package://hyq_description/meshes/sensors/vislab_3dve.stl"/>
+					<mesh filename="package://hyq2max_description/meshes/sensors/vislab_3dve.stl"/>
 				</geometry>
 			</collision>

Commit message: Corrected IMU origin position

File: robots/hyq2max.urdf.xacro (robot description, xacro)
@@ -78,5 +78,5 @@
 		accel_bias_mean="0.002"
 		accel_bias_stddev="0.001">
-		<origin xyz="0.3 0 0.095" rpy="0 ${-PI} 0"/>
+		<origin xyz="0.005 0 0.00125" rpy="0 ${-PI} 0"/>
 	</xacro:microstrain_3dmgx425_imu>
 	<!-- Velodyne -->

Commit message: [feature] Defined from an argument the enabling of joint sensors
The joint sensors measure the internal wrench of that joint

File: robots/hyq2max.urdf.xacro (robot description, xacro)
@@ -1,4 +1,6 @@
 <?xml version="1.0"?>
 <robot name="hyq2max" xmlns:xacro="http://www.ros.org/wiki/xacro">
+	<!-- This argument allows us to load joint sensors that measure the internal wrenches -->
+	<xacro:arg name="load_force_sensors" default="false"/>
 	<!-- The following included files set up definitions of parts of the robot body -->
 	<xacro:include filename="$(find hyq2max_description)/urdfs/common.xacro"/>
@@ -35,5 +37,6 @@
 		parent="trunk"
 		reflect_left="1"
-		reflect_front="1">
+		reflect_front="1"
+		load_force_sensors="$(arg load_force_sensors)">
 		<origin xyz="0.4435 0.097 0" rpy="${PI} ${PI/2} 0"/>
 <!--		<origin xyz="${d_fh/2} ${d_lr/2} 0" rpy="0 ${PI/2} ${PI}"/>-->
@@ -44,5 +47,6 @@
 		parent="trunk"
 		reflect_left="-1"
-		reflect_front="1">
+		reflect_front="1"
+		load_force_sensors="$(arg load_force_sensors)">
 		<origin xyz="0.4435 -0.097 0" rpy="0 ${PI/2} 0"/>
 <!--		<origin xyz="${d_fh/2} ${-d_lr/2} 0" rpy="0 ${PI/2} 0"/>-->
@@ -53,5 +57,6 @@
 		parent="trunk"
 		reflect_left="1"
-		reflect_front="-1">
+		reflect_front="-1"
+		load_force_sensors="$(arg load_force_sensors)">
 		<origin xyz="-0.4435 0.097 0" rpy="${PI} ${PI/2} 0"/>
 	</xacro:hyq2max_leg>
@@ -61,5 +66,6 @@
 		parent="trunk"
 		reflect_left="-1"
-		reflect_front="-1">
+		reflect_front="-1"
+		load_force_sensors="$(arg load_force_sensors)">
 		<origin xyz="-0.4435 -0.097 0" rpy="0 ${PI/2} 0"/>
 	</xacro:hyq2max_leg>

File: robots/hyq2max_model.urdf.xacro (robot description, xacro)
@@ -27,5 +27,6 @@
 		parent="trunk"
 		reflect_left="1"
-		reflect_front="1">
+		reflect_front="1"
+		load_force_sensors="false">
 		<origin xyz="0.4435 0.097 0" rpy="${PI} ${PI/2} 0"/>
 <!--		<origin xyz="${d_fh/2} ${d_lr/2} 0" rpy="0 ${PI/2} ${PI}"/>-->
@@ -36,5 +37,6 @@
 		parent="trunk"
 		reflect_left="-1"
-		reflect_front="1">
+		reflect_front="1"
+		load_force_sensors="false">
 		<origin xyz="0.4435 -0.097 0" rpy="0 ${PI/2} 0"/>
 <!--		<origin xyz="${d_fh/2} ${-d_lr/2} 0" rpy="0 ${PI/2} 0"/>-->
@@ -45,5 +47,6 @@
 		parent="trunk"
 		reflect_left="1"
-		reflect_front="-1">
+		reflect_front="-1"
+		load_force_sensors="false">
 		<origin xyz="-0.4435 0.097 0" rpy="${PI} ${PI/2} 0"/>
 	</xacro:hyq2max_leg>
@@ -53,5 +56,6 @@
 		parent="trunk"
 		reflect_left="-1"
-		reflect_front="-1">
+		reflect_front="-1"
+		load_force_sensors="false">
 		<origin xyz="-0.4435 -0.097 0" rpy="0 ${PI/2} 0"/>
 	</xacro:hyq2max_leg>

File: urdfs/leg/leg.gazebo.xacro (robot description, xacro)
@@ -1,5 +1,44 @@
 <?xml version="1.0"?>
 <robot xmlns:xacro="http://www.ros.org/wiki/xacro">
-	<xacro:macro name="leg_gazebo" params="name">
+	<xacro:macro name="leg_gazebo" params="name load_force_sensors">
+		<gazebo reference="${name}_haa_joint">
+			<provideFeedback>true</provideFeedback>
+		</gazebo>
+		<xacro:if value="${load_force_sensors}">
+			<gazebo>
+				<plugin name="${name}_haa_sensor" filename="libgazebo_ros_ft_sensor.so">
+					<robotNamespace>/hyq2max/internal_wrench/</robotNamespace>
+					<updateRate>100.0</updateRate>
+					<topicName>${name}_haa_joint</topicName>
+					<jointName>${name}_haa_joint</jointName>
+				</plugin>
+			</gazebo>
+		</xacro:if>
+		<gazebo reference="${name}_kfe_joint">
+			<provideFeedback>true</provideFeedback>
+		</gazebo>
+		<xacro:if value="${load_force_sensors}">
+			<gazebo>
+				<plugin name="${name}_kfe_sensor" filename="libgazebo_ros_ft_sensor.so">
+					<robotNamespace>/hyq2max/internal_wrench/</robotNamespace>
+					<updateRate>100.0</updateRate>
+					<topicName>${name}_kfe_joint</topicName>
+					<jointName>${name}_kfe_joint</jointName>
+				</plugin>
+			</gazebo>
+		</xacro:if>
+		<gazebo reference="${name}_hfe_joint">
+			<provideFeedback>true</provideFeedback>
+		</gazebo>
+		<xacro:if value="${load_force_sensors}">
+			<gazebo>
+				<plugin name="${name}_hfe_sensor" filename="libgazebo_ros_ft_sensor.so">
+					<robotNamespace>/hyq2max/internal_wrench/</robotNamespace>
+					<updateRate>100.0</updateRate>
+					<topicName>${name}_hfe_joint</topicName>
+					<jointName>${name}_hfe_joint</jointName>
+				</plugin>
+			</gazebo>
+		</xacro:if>
 		<gazebo reference="${name}_upperleg">
 			<kp>1000000.0</kp>

File: urdfs/leg/leg.urdf.xacro (robot description, xacro)
@@ -6,5 +6,5 @@
 	<!-- ================================== Leg ================================== -->
 	<!-- The xacro macro xacro:hyq2max_leg contains: hip assembly, upper and lower leg -->
-	<xacro:macro name="hyq2max_leg" params="name parent *origin reflect_left reflect_front">
+	<xacro:macro name="hyq2max_leg" params="name parent *origin reflect_left reflect_front load_force_sensors">
 		<!-- Joints -->
 		<!-- HAA joint -->
@@ -138,5 +138,5 @@
 		<!-- Extensions -->
 		<xacro:leg_transmission name="${name}"/>
-		<xacro:leg_gazebo name="${name}"/>
+		<xacro:leg_gazebo name="${name}" load_force_sensors="${load_force_sensors}"/>
 	</xacro:macro>
 </robot>

Commit message: parameterised details for gazebo

File: robots/hyq2max.urdf.xacro (robot description, xacro)
@@ -40,6 +40,6 @@
 		reflect_front="1"
 		load_force_sensors="$(arg load_force_sensors)">
-		<origin xyz="0.4435 0.097 0" rpy="${PI} ${PI/2} 0"/>
-<!--		<origin xyz="${d_fh/2} ${d_lr/2} 0" rpy="0 ${PI/2} ${PI}"/>-->
+		<!-- <origin xyz="0.4435 0.097 0" rpy="${PI} ${PI/2} 0"/>  -->
+		<origin xyz="${haa_fh/2} ${haa_lr/2} 0" rpy="${PI} ${PI/2} 0"/>
 	</xacro:hyq2max_leg>
 	<!-- RF leg -->
@@ -50,6 +50,6 @@
 		reflect_front="1"
 		load_force_sensors="$(arg load_force_sensors)">
-		<origin xyz="0.4435 -0.097 0" rpy="0 ${PI/2} 0"/>
-<!--		<origin xyz="${d_fh/2} ${-d_lr/2} 0" rpy="0 ${PI/2} 0"/>-->
+		<!-- <origin xyz="0.4435 -0.097 0" rpy="0 ${PI/2} 0"/> -->
+		<origin xyz="${haa_fh/2} ${-haa_lr/2} 0" rpy="0 ${PI/2} 0"/>
 	</xacro:hyq2max_leg>
 	<!-- LH leg -->
@@ -60,5 +60,6 @@
 		reflect_front="-1"
 		load_force_sensors="$(arg load_force_sensors)">
-		<origin xyz="-0.4435 0.097 0" rpy="${PI} ${PI/2} 0"/>
+		<!-- <origin xyz="-0.4435 0.097 0" rpy="${PI} ${PI/2} 0"/>  -->
+		<origin xyz="${-haa_fh/2} ${haa_lr/2} 0" rpy="${PI} ${PI/2} 0"/>
 	</xacro:hyq2max_leg>
 	<!-- RH leg -->
@@ -69,5 +70,6 @@
 		reflect_front="-1"
 		load_force_sensors="$(arg load_force_sensors)">
-		<origin xyz="-0.4435 -0.097 0" rpy="0 ${PI/2} 0"/>
+		<!-- <origin xyz="-0.4435 -0.097 0" rpy="0 ${PI/2} 0"/> -->
+		<origin xyz="${-haa_fh/2} ${-haa_lr/2} 0" rpy="0 ${PI/2} 0"/>
 	</xacro:hyq2max_leg>
 	<!-- IMU trunk -->

File: robots/hyq2max_model.urdf.xacro (robot description, xacro)
@@ -29,6 +29,6 @@
 		reflect_front="1"
 		load_force_sensors="false">
-		<origin xyz="0.4435 0.097 0" rpy="${PI} ${PI/2} 0"/>
-<!--		<origin xyz="${d_fh/2} ${d_lr/2} 0" rpy="0 ${PI/2} ${PI}"/>-->
+		<!-- <origin xyz="0.4435 0.097 0" rpy="${PI} ${PI/2} 0"/>  -->
+		<origin xyz="${haa_fh/2} ${haa_lr/2} 0" rpy="${PI} ${PI/2} 0"/>
 	</xacro:hyq2max_leg>
 	<!-- RF leg -->
@@ -39,6 +39,6 @@
 		reflect_front="1"
 		load_force_sensors="false">
-		<origin xyz="0.4435 -0.097 0" rpy="0 ${PI/2} 0"/>
-<!--		<origin xyz="${d_fh/2} ${-d_lr/2} 0" rpy="0 ${PI/2} 0"/>-->
+		<!-- <origin xyz="0.4435 -0.097 0" rpy="0 ${PI/2} 0"/> -->
+		<origin xyz="${haa_fh/2} ${-haa_lr/2} 0" rpy="0 ${PI/2} 0"/>
 	</xacro:hyq2max_leg>
 	<!-- LH leg -->
@@ -49,5 +49,6 @@
 		reflect_front="-1"
 		load_force_sensors="false">
-		<origin xyz="-0.4435 0.097 0" rpy="${PI} ${PI/2} 0"/>
+		<!-- <origin xyz="-0.4435 0.097 0" rpy="${PI} ${PI/2} 0"/>  -->
+		<origin xyz="${-haa_fh/2} ${haa_lr/2} 0" rpy="${PI} ${PI/2} 0"/>
 	</xacro:hyq2max_leg>
 	<!-- RH leg -->
@@ -58,5 +59,6 @@
 		reflect_front="-1"
 		load_force_sensors="false">
-		<origin xyz="-0.4435 -0.097 0" rpy="0 ${PI/2} 0"/>
+		<!-- <origin xyz="-0.4435 -0.097 0" rpy="0 ${PI/2} 0"/> -->
+		<origin xyz="${-haa_fh/2} ${-haa_lr/2} 0" rpy="0 ${PI/2} 0"/>
 	</xacro:hyq2max_leg>
 </robot>

File: urdfs/common.xacro (robot description, xacro)
@@ -3,6 +3,10 @@
 	<property name="PI" value="3.1415926535897931"/>
 	<!-- standard distances -->
-	<property name="d_lr" value="0.414"/>
-	<property name="d_fh" value="0.747"/>
+	<property name="d_lr" value="0.7245"/>
+	<property name="d_fh" value="1.1952"/>
+	<property name="haa_lr" value="0.34125"/>
+	<!-- 0.194  0.34125 -->
+	<property name="haa_fh" value="1.4192"/>
+	<!-- 0.887 1.4192-->
 	<property name="hipassembly_length" value="0.117"/>
 	<property name="upperleg_length" value="0.360"/>
@@ -15,11 +19,11 @@
 	<property name="ycom_trunk" value="0.000598"/>
 	<property name="zcom_trunk" value="-0.007592"/>
-	<property name="m_trunk" value="39.71"/>
-	<property name="ixx_trunk" value="0.3020795"/>
-	<property name="iyy_trunk" value="4.751448"/>
-	<property name="izz_trunk" value="4.82415"/>
-	<property name="ixy_trunk" value="-0.0050854"/>
-	<property name="ixz_trunk" value="0.0046576"/>
-	<property name="iyz_trunk" value="-0.0017613"/>
+	<property name="m_trunk" value="79.71"/>
+	<property name="ixx_trunk" value="1.620351283145943"/>
+	<property name="iyy_trunk" value="23.421032273196097"/>
+	<property name="izz_trunk" value="25.933247447558614"/>
+	<property name="ixy_trunk" value="-0.028582227529590"/>
+	<property name="ixz_trunk" value="0.014958742724754"/>
+	<property name="iyz_trunk" value="-0.006187059688995"/>
 	<!-- Hip assembly -->
 	<property name="xcom_hipassembly" value="-0.000605"/>

Commit message: [wip] Added the multisense sensor

File: robots/hyq2max.urdf.xacro (robot description, xacro)
@@ -18,4 +18,5 @@
 	<xacro:include filename="$(find sensors_description)/urdfs/sensors/bumblebee.urdf.xacro"/>
 	<xacro:include filename="$(find sensors_description)/urdfs/sensors/vislab_3dve.urdf.xacro"/>
+	<xacro:include filename="$(find sensors_description)/urdfs/sensors/multisense_sl.urdf.xacro"/>
 	<!-- Generic simulator_gazebo plugins for starting mechanism control, ros time -->
 	<xacro:include filename="$(find hyq2max_description)/gazebo/gazebo.urdf.xacro"/>
@@ -119,3 +120,6 @@
 		rpy="0 0 0"
 		high_res="false"/>-->
+        <xacro:multisense_sl parent="trunk" prefix="hyq">
+            <origin xyz="0.701737 0.0 -0.05" rpy="-0.0241345 0.446222 -0.0347202"/>
+        </xacro:multisense_sl>
 </robot>

Commit message: Compliance with new xacro

File: robots/hyq2max.urdf.xacro (robot description, xacro)
@@ -31,5 +31,5 @@
 	<!-- Trunk -->
 	<xacro:hyq2max_trunk name="base">
-		<origin xyz="-0.443 -0.191 -0.276" rpy="0 0 0"/>
+		<!-- <origin xyz="-0.443 -0.191 -0.276" rpy="0 0 0"/> -->
 	</xacro:hyq2max_trunk>
 	<!-- LF leg -->

File: robots/hyq2max_model.urdf.xacro (robot description, xacro)
@@ -20,5 +20,5 @@
 	<!-- Trunk -->
 	<xacro:hyq2max_trunk name="base">
-		<origin xyz="-0.443 -0.191 -0.276" rpy="0 0 0"/>
+		<!-- <origin xyz="-0.443 -0.191 -0.276" rpy="0 0 0"/> -->
 	</xacro:hyq2max_trunk>
 	<!-- LF leg -->

File: urdfs/common.xacro (robot description, xacro)
@@ -1,4 +1,4 @@
 <?xml version="1.0"?>
-<robot>
+<robot xmlns:xacro="http://ros.org/wiki/xacro">
 	<xacro:property name="PI" value="3.1415926535897931"/>
 	<!-- standard distances -->

File: urdfs/leg/leg.urdf.xacro (robot description, xacro)
@@ -39,9 +39,9 @@
 			<dynamics damping="0.1" friction="0" />
             <limit effort="250.0" velocity="12.0"
-                   lower="${(1-reflect_front)*2*PI/180-(1+reflect_front)*167*PI/180}"
-                   upper="${-(1+reflect_front)*2*PI/180+(1-reflect_front)*167*PI/180}"/>
+                   lower="${(1-reflect_front)*2*PI/360-(1+reflect_front)*167*PI/360}"
+                   upper="${-(1+reflect_front)*2*PI/360+(1-reflect_front)*167*PI/360}"/>
             <safety_controller k_position="100" k_velocity="100"
-                               soft_lower_limit="${(1-reflect_front)*2*PI/180-(1+reflect_front)*167*PI/180}"
-                               soft_upper_limit="${-(1+reflect_front)*2*PI/180+(1-reflect_front)*167*PI/180}" />
+                               soft_lower_limit="${(1-reflect_front)*2*PI/360-(1+reflect_front)*167*PI/360}"
+                               soft_upper_limit="${-(1+reflect_front)*2*PI/360+(1-reflect_front)*167*PI/360}" />
 		</joint>
 		<!-- Foot joint -->

Commit message: Removing unused vision sensors

File: robots/hyq2max.urdf.xacro (robot description, xacro)
@@ -13,8 +13,4 @@
 	<xacro:include filename="$(find sensors_description)/urdfs/sensors/microstrain_3dmgx425_imu.urdf.xacro"/>
 	<xacro:include filename="$(find sensors_description)/urdfs/sensors/asus_xtion.urdf.xacro"/>
-	<xacro:include filename="$(find sensors_description)/urdfs/sensors/velodyne.urdf.xacro"/>
-	<xacro:include filename="$(find sensors_description)/urdfs/sensors/kinect.urdf.xacro"/>
-	<xacro:include filename="$(find sensors_description)/urdfs/sensors/ptu_d46.urdf.xacro"/>
-	<xacro:include filename="$(find sensors_description)/urdfs/sensors/bumblebee.urdf.xacro"/>
 	<xacro:include filename="$(find sensors_description)/urdfs/sensors/vislab_3dve.urdf.xacro"/>
 	<!-- Generic simulator_gazebo plugins for starting mechanism control, ros time -->
@@ -81,16 +77,4 @@
 		<origin xyz="0.005 0 0.00125" rpy="0 ${-PI} 0"/>
 	</xacro:microstrain_3dmgx425_imu>
-	<!-- Velodyne -->
-<!--	<xacro:velodyne
-		name="trunk_mount"
-		parent="trunk">
-		<origin xyz="0.39 0 0.269" rpy="0 0 0"/>
-	</xacro:velodyne>-->
-	<!-- PTU unit -->
-<!--	<xacro:ptu_d46
-		name="ptu"
-		parent="trunk">
-		<origin xyz="0.657353 0.015447 0.119533" rpy="-0.013127 0.569257 -0.007748"/>
-	</xacro:ptu_d46>-->
 	<!-- Asus Xtion Pro -->
 	<!--<origin xyz="0 0.005 0.036" rpy="0 0 0"/> with Bumblebee setup -->
@@ -101,18 +85,4 @@
 		<origin xyz="0 0.005 0.036" rpy="0 0 0"/>
 	</xacro:asus_xtion_camera>-->
-	<!-- Kinect --> <!-- is no more used, but we keep it for compatibilty -->
-	<!--xacro:kinect_camera
-		name="head_mount"
-		parent="trunk">
-		<origin xyz="0.63 0 0.095" rpy="0 0 0"/>
-	</xacro:kinect_camera-->
-	<!-- Bumblebee -->
-<!--	<xacro:bumblebee_97
-		parent_link="ptu_mount_link"
-		xyz="0 0 0.018"
-		rpy="0 0 0"
-		ns="bumblebee"
-		frame_prefix="bumblebee_"
-		high_res="false"/>-->
 <!--	<xacro:vislab_3dve_72
 		name="vislab_3dve"
